Commit message: second turtorial updates

File: interbotix_xsarm_descriptions/urdf/ur5robot.urdf (robot description, URDF)
Before this commit: robot universal-robot-ur5, 15 links, 14 joints
Links:
- added link rear_camera_link, mass 0.1; collision box size=0.1 0.1 0.1; visual box size=0.1 0.1 0.1
Joints:
- added joint rear_camera_joint: type fixed, parent world, child rear_camera_link, origin xyz=-1.0 0 1.8 rpy=0 0.2967 0

File: ur5_moveit/config/gazebo_universal-robot-ur5.urdf (robot description, URDF)
Before this commit: robot universal-robot-ur5, 15 links, 14 joints
Links:
- added link rear_camera_link; visual box size=0.1 0.1 0.1
Joints:
- added joint rear_camera_joint: type fixed, parent world, child rear_camera_link, origin xyz=-0.3 0 1.5 rpy=0 0.083 0

Commit message: Final Updates

File: interbotix_xsarm_descriptions/urdf/ur5robot.urdf (robot description, URDF)
Before this commit: robot universal-robot-ur5, 16 links, 15 joints
Joints:
- joint left_inner_finger_joint: mimic joint=finger_joint multiplier=1 offset=0 -> (none)
- joint left_inner_knuckle_joint: mimic joint=finger_joint multiplier=-1 offset=0 -> (none)
- joint right_inner_finger_joint: mimic joint=finger_joint multiplier=1 offset=0 -> (none)
- joint right_inner_knuckle_joint: mimic joint=finger_joint multiplier=-1 offset=0 -> (none)
- joint right_outer_knuckle_joint: mimic joint=finger_joint multiplier=-1 offset=0 -> (none)
